Commit message: Phase 1.1: realign layout to EstacionMezzanine.dxf
DXF (mm, INSUNITS=4) is now the source of truth for all planar XY positions.
Z values come from prior physical measurements or component specs where the
DXF does not provide height. Origin convention (table LL corner) unchanged.

Layout changes:
- conveyor: pos (0.500,0.300)->(0.385,0.302); size 0.400x0.132x0.055 ->
  0.700x0.215x0.060 (DOBOT Conveyor Belt Kit official).
- cube_base: pos (0.110,0.030)->(0.020,0.348); now upper-left of cobot.
- cubes: single demo cube replaced with 3x3 grid of 9 color-differentiated
  cubes (red/green/blue/yellow/orange/white/magenta/cyan/dark_gray) +
  5 mm reborde frame on the base.
- hmi: pos (0.650,0.425)->(0.650,0.517) (between conveyor back edge and
  PLC cabinet); base footprint 0.140x0.060 -> 0.168x0.067 per DXF.
- computer: pos (1.250,0.030)->(1.137,0.260); footprint now 0.372x0.432
  (full workstation area, extends past table edges). Tower (Lenovo tinker
  bbox 0.11825x0.07239x0.0861) at back-right; monitor + keyboard + mouse
  placeholders in front.
- photoelectric_sensor: local (0.210,0.120,0.050)->(0.217,0.218,0.060);
  now at back edge of conveyor per DXF U-shape bracket.
- camera_profile: column profile_x 0.690->0.598; arm length 0.316->0.169
  (exact recompute) so camera body centers over DXF orange footprint
  (0.618, 0.407, 0.635). Z kept from Phase 1.
- white_board: pos (0.090,0.035)->(0.109,0.034); kept as flat plate.
- cobot_base, plc_cabinet, buttons_panel: XY unchanged (DXF confirms).

New: explicit start_button (r=0.019) and emergency_stop_button (r=0.029)
positions per DXF circles. Materials add mz_magenta, mz_cyan,
mz_cube_base_brown.

Added reference/dxf/EstacionMezzanine.dxf and reference/rviz_screenshots/
phase_1_1_dxf_driven.png. docs/measurements.md gains the color-to-component
map and a Phase 1 -> 1.1 delta table; docs/validation.md updated with the
new expected coordinates.

Co-Authored-By: Claude Opus 4.7 (1M context) <noreply@anthropic.com>

File: mezzanine_rviz_sim/urdf/buttons_panel.xacro (robot description, xacro)
@@ -2,13 +2,17 @@
 <robot xmlns:xacro="http://ros.org/wiki/xacro">
   <!--
-    Start + Emergency Stop panel.
-    Panel placeholder size 0.10 x 0.15 x 0.05 m (TBD).
-    Position xyz = (1.170, 0.040, 0) m is the lower-left-front corner.
-    Two cylindrical buttons mounted on TOP face: green Start and red E-Stop.
+    Start + Emergency Stop panel (cyan rectangle in EstacionMezzanine.dxf).
+    Panel size 0.10 x 0.15 x 0.05 m. Position xyz = (1.170, 0.040, 0) m is
+    the lower-left-front corner. Two cylindrical buttons mounted on TOP face:
+      - green Start: DXF circle r=0.019 m at world (1.220, 0.072).
+        Local on panel TOP: (0.050, 0.032).
+      - red E-Stop (mushroom): DXF circle r=0.029 m at world (1.220, 0.146).
+        Local on panel TOP: (0.050, 0.106).
   -->
   <xacro:property name="panel_size_x" value="0.100"/>
   <xacro:property name="panel_size_y" value="0.150"/>
   <xacro:property name="panel_size_z" value="0.050"/>
-  <xacro:property name="btn_radius" value="0.020"/>
+  <xacro:property name="start_btn_radius" value="0.019"/>
+  <xacro:property name="estop_btn_radius" value="0.029"/>
   <xacro:property name="btn_height" value="0.012"/>
   <xacro:macro name="mz_buttons_panel" params="parent:=table_origin x:=1.170 y:=0.040 z:=0.000">
@@ -37,5 +41,5 @@
         <origin xyz="0 0 ${btn_height/2}" rpy="0 0 0"/>
         <geometry>
-          <cylinder radius="${btn_radius}" length="${btn_height}"/>
+          <cylinder radius="${start_btn_radius}" length="${btn_height}"/>
         </geometry>
         <material name="mz_green"/>
@@ -44,5 +48,5 @@
         <origin xyz="0 0 ${btn_height/2}" rpy="0 0 0"/>
         <geometry>
-          <cylinder radius="${btn_radius}" length="${btn_height}"/>
+          <cylinder radius="${start_btn_radius}" length="${btn_height}"/>
         </geometry>
       </collision>
@@ -51,5 +55,5 @@
       <parent link="start_button_panel"/>
       <child link="start_button"/>
-      <origin xyz="${panel_size_x/2} ${panel_size_y*0.3} ${panel_size_z}" rpy="0 0 0"/>
+      <origin xyz="0.050 0.032 ${panel_size_z}" rpy="0 0 0"/>
     </joint>
     <link name="emergency_stop_button">
@@ -57,5 +61,5 @@
         <origin xyz="0 0 ${btn_height/2}" rpy="0 0 0"/>
         <geometry>
-          <cylinder radius="${btn_radius}" length="${btn_height}"/>
+          <cylinder radius="${estop_btn_radius}" length="${btn_height}"/>
         </geometry>
         <material name="mz_red"/>
@@ -64,5 +68,5 @@
         <origin xyz="0 0 ${btn_height/2}" rpy="0 0 0"/>
         <geometry>
-          <cylinder radius="${btn_radius}" length="${btn_height}"/>
+          <cylinder radius="${estop_btn_radius}" length="${btn_height}"/>
         </geometry>
       </collision>
@@ -71,5 +75,5 @@
       <parent link="start_button_panel"/>
       <child link="emergency_stop_button"/>
-      <origin xyz="${panel_size_x/2} ${panel_size_y*0.7} ${panel_size_z}" rpy="0 0 0"/>
+      <origin xyz="0.050 0.106 ${panel_size_z}" rpy="0 0 0"/>
     </joint>
   </xacro:macro>

File: mezzanine_rviz_sim/urdf/camera_frame.xacro (robot description, xacro)
@@ -3,7 +3,12 @@
   <!--
     Camera support: vertical aluminum profile (4x4 cm cross section) standing
-    at sensor xy with height 0.720 m (TBD placeholder), plus a horizontal arm
-    extending in -y to support the camera. Camera placed at the documented
-    position (0.595, 0.260, 0.635) m.
+    at LL=(0.598, 0.556) m (pegada a la cabina - back edge at y=0.596),
+    with a horizontal arm extending in -y to support the camera.
+    DXF source: orange RGB 248,153,30 rectangle (camera body footprint
+    centered at (0.618, 0.407)).
+    Geometry: camera_world_y = profile_y + cs_y/2 - arm_len_y. With
+    profile_y=0.556, cs_y/2=0.020 and camera_y=0.407, arm_len_y=0.169 m
+    (computed exact instead of 0.189 m estimate from the diagnostic).
+    Z=0.635 m kept from Phase 1; the DXF only provides planar XY.
   -->
   <xacro:property name="profile_cs_x" value="0.040"/>
@@ -14,7 +19,7 @@
   <xacro:property name="camera_size_z" value="0.060"/>
   <xacro:macro name="mz_camera_support" params="parent:=table_origin
-                                                 profile_x:=0.575
-                                                 profile_y:=0.400
-                                                 profile_arm_len_y:=0.180
+                                                 profile_x:=0.598
+                                                 profile_y:=0.556
+                                                 profile_arm_len_y:=0.169
                                                  camera_z:=0.635">
     <link name="camera_profile">

File: mezzanine_rviz_sim/urdf/computer.xacro (robot description, xacro)
@@ -2,29 +2,67 @@
 <robot xmlns:xacro="http://ros.org/wiki/xacro">
   <!--
-    Computer placeholder on the RIGHT side of the table.
-    Position xyz = lower-left-front corner of the workstation footprint.
-    Workstation = a vertical tower (black box) + a flat monitor with stand.
-    Dimensions are placeholders (TBD - to confirm against photos).
+    Computer workstation - visual approximation of the full computer area.
+    The magenta rectangle in EstacionMezzanine.dxf is the FULL workstation
+    footprint (372 x 432 mm), NOT just the tower. It represents tower +
+    monitor + keyboard + mouse and extends past the table edges.
+    Position from DXF: workstation LL = (1.137, 0.260, 0) m.
+    Tower model: Lenovo IdeaCentre / tinker. Bounding box from tinker.obj:
+      0.11825 x 0.07239 x 0.0861 m.
+    The tower is placed toward the BACK-RIGHT of the magenta footprint per
+    user direction. Remaining area is monitor (centered, with stand) and
+    a flat keyboard/mouse placeholder in front.
+    NOTE: VISUAL APPROXIMATION. The magenta footprint represents the entire
+    workstation, not just the tower. Collision boxes are simple primitives.
+    To swap the tower primitive for a tinker.obj mesh, stage the OBJ under
+    meshes/computer/tinker.obj and replace the tower <box> with:
+      <mesh filename="package://mezzanine_rviz_sim/meshes/computer/tinker.obj"
+            scale="0.001 0.001 0.001"/>
   -->
-  <xacro:property name="tower_size_x" value="0.090"/>
-  <xacro:property name="tower_size_y" value="0.230"/>
-  <xacro:property name="tower_size_z" value="0.380"/>
-  <xacro:property name="mon_stand_x" value="0.140"/>
-  <xacro:property name="mon_stand_y" value="0.180"/>
+  <!-- Workstation footprint (DXF magenta: 0.372 x 0.432) -->
+  <xacro:property name="ws_size_x" value="0.372"/>
+  <xacro:property name="ws_size_y" value="0.432"/>
+  <!-- Lenovo tinker tower bounding box (mm-to-m from tinker.obj) -->
+  <xacro:property name="tower_size_x" value="0.11825"/>
+  <xacro:property name="tower_size_y" value="0.07239"/>
+  <xacro:property name="tower_size_z" value="0.0861"/>
+  <!-- Tower local placement: back-right of workstation with 20 mm margin -->
+  <xacro:property name="tower_local_x" value="${ws_size_x - tower_size_x - 0.020}"/>
+  <xacro:property name="tower_local_y" value="${ws_size_y - tower_size_y - 0.020}"/>
+  <!-- Monitor stand (flat foot), centered in workstation X -->
+  <xacro:property name="mon_stand_x" value="0.180"/>
+  <xacro:property name="mon_stand_y" value="0.140"/>
   <xacro:property name="mon_stand_z" value="0.020"/>
+  <xacro:property name="mon_stand_local_x" value="${(ws_size_x - mon_stand_x) / 2}"/>
+  <xacro:property name="mon_stand_local_y" value="${ws_size_y - mon_stand_y - 0.060}"/>
+  <!-- Monitor riser / column -->
   <xacro:property name="mon_col_x" value="0.030"/>
   <xacro:property name="mon_col_y" value="0.030"/>
-  <xacro:property name="mon_col_z" value="0.090"/>
-  <xacro:property name="mon_size_x" value="0.450"/>
+  <xacro:property name="mon_col_z" value="0.110"/>
+  <!-- Monitor body and screen -->
+  <xacro:property name="mon_size_x" value="0.520"/>
   <xacro:property name="mon_size_y" value="0.030"/>
-  <xacro:property name="mon_size_z" value="0.260"/>
-  <xacro:property name="mon_scr_x" value="0.410"/>
-  <xacro:property name="mon_scr_y" value="0.004"/>
-  <xacro:property name="mon_scr_z" value="0.230"/>
-  <xacro:macro name="mz_computer" params="parent:=table_origin x:=1.250 y:=0.030 z:=0.000">
+  <xacro:property name="mon_size_z" value="0.310"/>
+  <xacro:property name="mon_scr_x"  value="0.480"/>
+  <xacro:property name="mon_scr_y"  value="0.004"/>
+  <xacro:property name="mon_scr_z"  value="0.280"/>
+  <!-- Keyboard placeholder (flat box) in front area -->
+  <xacro:property name="kbd_size_x" value="0.280"/>
+  <xacro:property name="kbd_size_y" value="0.110"/>
+  <xacro:property name="kbd_size_z" value="0.018"/>
+  <xacro:property name="kbd_local_x" value="${(ws_size_x - kbd_size_x) / 2}"/>
+  <xacro:property name="kbd_local_y" value="0.020"/>
+  <!-- Mouse placeholder -->
+  <xacro:property name="mouse_size_x" value="0.060"/>
+  <xacro:property name="mouse_size_y" value="0.100"/>
+  <xacro:property name="mouse_size_z" value="0.030"/>
+  <xacro:property name="mouse_local_x" value="${ws_size_x - mouse_size_x - 0.030}"/>
+  <xacro:property name="mouse_local_y" value="0.030"/>
+  <xacro:macro name="mz_computer" params="parent:=table_origin x:=1.137 y:=0.260 z:=0.000">
     <link name="computer">
-      <!-- Tower (CPU box, vertical) -->
+      <!-- Tower (Lenovo tinker visual approximation) -->
       <visual>
-        <origin xyz="${tower_size_x/2} ${tower_size_y/2} ${tower_size_z/2}" rpy="0 0 0"/>
+        <origin xyz="${tower_local_x + tower_size_x/2}
+                     ${tower_local_y + tower_size_y/2}
+                     ${tower_size_z/2}" rpy="0 0 0"/>
         <geometry>
           <box size="${tower_size_x} ${tower_size_y} ${tower_size_z}"/>
@@ -33,12 +71,16 @@
       </visual>
       <collision>
-        <origin xyz="${tower_size_x/2} ${tower_size_y/2} ${tower_size_z/2}" rpy="0 0 0"/>
+        <origin xyz="${tower_local_x + tower_size_x/2}
+                     ${tower_local_y + tower_size_y/2}
+                     ${tower_size_z/2}" rpy="0 0 0"/>
         <geometry>
           <box size="${tower_size_x} ${tower_size_y} ${tower_size_z}"/>
         </geometry>
       </collision>
-      <!-- Monitor stand -->
+      <!-- Monitor stand (flat foot) -->
       <visual>
-        <origin xyz="${tower_size_x + 0.020 + mon_stand_x/2} ${mon_stand_y/2 + 0.020} ${mon_stand_z/2}" rpy="0 0 0"/>
+        <origin xyz="${mon_stand_local_x + mon_stand_x/2}
+                     ${mon_stand_local_y + mon_stand_y/2}
+                     ${mon_stand_z/2}" rpy="0 0 0"/>
         <geometry>
           <box size="${mon_stand_x} ${mon_stand_y} ${mon_stand_z}"/>
@@ -46,8 +88,8 @@
         <material name="mz_dark_gray"/>
       </visual>
-      <!-- Monitor column (riser) -->
+      <!-- Monitor riser / column -->
       <visual>
-        <origin xyz="${tower_size_x + 0.020 + mon_stand_x/2}
-                     ${mon_stand_y/2 + 0.020}
+        <origin xyz="${mon_stand_local_x + mon_stand_x/2}
+                     ${mon_stand_local_y + mon_stand_y/2}
                      ${mon_stand_z + mon_col_z/2}" rpy="0 0 0"/>
         <geometry>
@@ -58,6 +100,6 @@
       <!-- Monitor body (bezel) -->
       <visual>
-        <origin xyz="${tower_size_x + 0.020 + mon_stand_x/2}
-                     ${mon_stand_y/2 + 0.020}
+        <origin xyz="${mon_stand_local_x + mon_stand_x/2}
+                     ${mon_stand_local_y + mon_stand_y/2}
                      ${mon_stand_z + mon_col_z + mon_size_z/2}" rpy="0 0 0"/>
         <geometry>
@@ -66,8 +108,8 @@
         <material name="mz_dark_gray"/>
       </visual>
-      <!-- Screen face on front (-y of monitor body) -->
+      <!-- Screen face on front (-y) -->
       <visual>
-        <origin xyz="${tower_size_x + 0.020 + mon_stand_x/2}
-                     ${mon_stand_y/2 + 0.020 - mon_size_y/2 - mon_scr_y/2}
+        <origin xyz="${mon_stand_local_x + mon_stand_x/2}
+                     ${mon_stand_local_y + mon_stand_y/2 - mon_size_y/2 - mon_scr_y/2}
                      ${mon_stand_z + mon_col_z + mon_size_z/2}" rpy="0 0 0"/>
         <geometry>
@@ -75,4 +117,24 @@
         </geometry>
         <material name="mz_hmi_dark"/>
+      </visual>
+      <!-- Keyboard placeholder -->
+      <visual>
+        <origin xyz="${kbd_local_x + kbd_size_x/2}
+                     ${kbd_local_y + kbd_size_y/2}
+                     ${kbd_size_z/2}" rpy="0 0 0"/>
+        <geometry>
+          <box size="${kbd_size_x} ${kbd_size_y} ${kbd_size_z}"/>
+        </geometry>
+        <material name="mz_dark_gray"/>
+      </visual>
+      <!-- Mouse placeholder -->
+      <visual>
+        <origin xyz="${mouse_local_x + mouse_size_x/2}
+                     ${mouse_local_y + mouse_size_y/2}
+                     ${mouse_size_z/2}" rpy="0 0 0"/>
+        <geometry>
+          <box size="${mouse_size_x} ${mouse_size_y} ${mouse_size_z}"/>
+        </geometry>
+        <material name="mz_dark_gray"/>
       </visual>
     </link>

File: mezzanine_rviz_sim/urdf/conveyor.xacro (robot description, xacro)
@@ -2,12 +2,15 @@
 <robot xmlns:xacro="http://ros.org/wiki/xacro">
   <!--
-    Conveyor. Width 0.132 m, thickness 0.055 m confirmed.
-    Length TBD - placeholder 0.400 m.
-    Position: lower-left-front corner at (0.385, 0.300, 0.000) m.
+    Conveyor.
+    Model: DOBOT Conveyor Belt Kit (official spec).
+    Official dimensions: 700 x 215 x 60 mm = 0.700 x 0.215 x 0.060 m.
+    Position (from EstacionMezzanine.dxf): table-frame LL corner = (0.385, 0.302, 0).
+    Notes: effective_travel ~= 0.600 m, payload 0.5 kg, max speed 0.120 m/s.
+    Official STEP/SolidWorks file not yet located (see layout_params.yaml).
   -->
-  <xacro:property name="conveyor_size_x" value="0.400"/>
-  <xacro:property name="conveyor_size_y" value="0.132"/>
-  <xacro:property name="conveyor_size_z" value="0.055"/>
-  <xacro:macro name="mz_conveyor" params="parent:=table_origin x:=0.385 y:=0.300 z:=0.000">
+  <xacro:property name="conveyor_size_x" value="0.700"/>
+  <xacro:property name="conveyor_size_y" value="0.215"/>
+  <xacro:property name="conveyor_size_z" value="0.060"/>
+  <xacro:macro name="mz_conveyor" params="parent:=table_origin x:=0.385 y:=0.302 z:=0.000">
     <link name="conveyor_base">
       <visual>

File: mezzanine_rviz_sim/urdf/cubes_and_base.xacro (robot description, xacro)
@@ -2,15 +2,47 @@
 <robot xmlns:xacro="http://ros.org/wiki/xacro">
   <!--
-    Cube base (blue fixture) + one demo cube.
-    Cube base: 0.140 x 0.140 x 0.020 m at (0.348, 0.020, 0) m (lower-left-front).
-    Cube_01: 0.040 x 0.040 x 0.050 m sitting on top of the cube base, centered.
+    Cube base + 9 cubes in a 3x3 grid.
+    Positions and counts come from EstacionMezzanine.dxf:
+      - base (orange RGB 205,105,40): outer 140x140 mm, inner 130x130 mm
+        (5 mm reborde / lip) at table-frame LL=(0.020, 0.348).
+      - 9 cubes (yellow in DXF): 40x40x40 footprint, grid 3x3, centered on base.
+    Local layout in cube_base frame:
+      - base LL at (0,0,0), size 0.140 x 0.140 x 0.020.
+      - 5 mm lip occupies the outer 5 mm; cube grid spans local
+        (0.010, 0.010) to (0.130, 0.130).
+      - cube[i][j] LL local = (0.010 + j*0.040, 0.010 + i*0.040, 0.020).
+    Cubes are color-differentiated for clarity (mz_red, mz_green, mz_blue,
+    mz_yellow, mz_orange, mz_white, mz_magenta, mz_cyan, mz_dark_gray).
   -->
   <xacro:property name="cube_base_size_x" value="0.140"/>
   <xacro:property name="cube_base_size_y" value="0.140"/>
   <xacro:property name="cube_base_size_z" value="0.020"/>
-  <xacro:property name="cube_size_x" value="0.040"/>
-  <xacro:property name="cube_size_y" value="0.040"/>
-  <xacro:property name="cube_size_z" value="0.050"/>
-  <xacro:macro name="mz_cube_base" params="parent:=table_origin x:=0.348 y:=0.020 z:=0.000">
+  <xacro:property name="cube_base_lip"    value="0.005"/>
+  <xacro:property name="lip_h"            value="0.005"/>
+  <xacro:property name="cube_size" value="0.040"/>
+  <xacro:macro name="mz_cube" params="name x_local y_local z_local material">
+    <link name="${name}">
+      <visual>
+        <origin xyz="${cube_size/2} ${cube_size/2} ${cube_size/2}" rpy="0 0 0"/>
+        <geometry>
+          <box size="${cube_size} ${cube_size} ${cube_size}"/>
+        </geometry>
+        <material name="${material}"/>
+      </visual>
+      <collision>
+        <origin xyz="${cube_size/2} ${cube_size/2} ${cube_size/2}" rpy="0 0 0"/>
+        <geometry>
+          <box size="${cube_size} ${cube_size} ${cube_size}"/>
+        </geometry>
+      </collision>
+    </link>
+    <joint name="cube_base_to_${name}" type="fixed">
+      <parent link="cube_base"/>
+      <child link="${name}"/>
+      <origin xyz="${x_local} ${y_local} ${z_local}" rpy="0 0 0"/>
+    </joint>
+  </xacro:macro>
+  <xacro:macro name="mz_cube_base" params="parent:=table_origin x:=0.020 y:=0.348 z:=0.000">
+    <!-- Base body (orange RGB 205,105,40 per DXF) -->
     <link name="cube_base">
       <visual>
@@ -19,5 +51,5 @@
           <box size="${cube_base_size_x} ${cube_base_size_y} ${cube_base_size_z}"/>
         </geometry>
-        <material name="mz_blue"/>
+        <material name="mz_cube_base_brown"/>
       </visual>
       <collision>
@@ -33,24 +65,57 @@
       <origin xyz="${x} ${y} ${z}" rpy="0 0 0"/>
     </joint>
-    <link name="cube_01">
+    <!--
+      5 mm reborde: thin frame around the inner pocket on top of the base.
+      Visual hint only; collision stays the base block.
+    -->
+    <link name="cube_base_lip">
       <visual>
-        <origin xyz="${cube_size_x/2} ${cube_size_y/2} ${cube_size_z/2}" rpy="0 0 0"/>
+        <origin xyz="${cube_base_size_x/2} ${cube_base_lip/2} ${cube_base_size_z + lip_h/2}" rpy="0 0 0"/>
         <geometry>
-          <box size="${cube_size_x} ${cube_size_y} ${cube_size_z}"/>
+          <box size="${cube_base_size_x} ${cube_base_lip} ${lip_h}"/>
         </geometry>
-        <material name="mz_orange"/>
+        <material name="mz_cube_base_brown"/>
       </visual>
-      <collision>
-        <origin xyz="${cube_size_x/2} ${cube_size_y/2} ${cube_size_z/2}" rpy="0 0 0"/>
+      <visual>
+        <origin xyz="${cube_base_size_x/2} ${cube_base_size_y - cube_base_lip/2} ${cube_base_size_z + lip_h/2}" rpy="0 0 0"/>
         <geometry>
-          <box size="${cube_size_x} ${cube_size_y} ${cube_size_z}"/>
+          <box size="${cube_base_size_x} ${cube_base_lip} ${lip_h}"/>
         </geometry>
-      </collision>
+        <material name="mz_cube_base_brown"/>
+      </visual>
+      <visual>
+        <origin xyz="${cube_base_lip/2} ${cube_base_size_y/2} ${cube_base_size_z + lip_h/2}" rpy="0 0 0"/>
+        <geometry>
+          <box size="${cube_base_lip} ${cube_base_size_y} ${lip_h}"/>
+        </geometry>
+        <material name="mz_cube_base_brown"/>
+      </visual>
+      <visual>
+        <origin xyz="${cube_base_size_x - cube_base_lip/2} ${cube_base_size_y/2} ${cube_base_size_z + lip_h/2}" rpy="0 0 0"/>
+        <geometry>
+          <box size="${cube_base_lip} ${cube_base_size_y} ${lip_h}"/>
+        </geometry>
+        <material name="mz_cube_base_brown"/>
+      </visual>
     </link>
-    <joint name="cube_base_to_cube_01" type="fixed">
+    <joint name="cube_base_to_cube_base_lip" type="fixed">
       <parent link="cube_base"/>
-      <child link="cube_01"/>
-      <origin xyz="${cube_base_size_x/2 - cube_size_x/2} ${cube_base_size_y/2 - cube_size_y/2} ${cube_base_size_z}" rpy="0 0 0"/>
+      <child link="cube_base_lip"/>
+      <origin xyz="0 0 0" rpy="0 0 0"/>
     </joint>
+    <!--
+      3x3 grid of 40 mm cubes. Row index i (0..2) increases in +y;
+      column index j (0..2) increases in +x. Grid origin local to
+      cube_base: (0.010, 0.010, 0.020). Cubes are color-differentiated.
+    -->
+    <xacro:mz_cube name="cube_00" x_local="0.010" y_local="0.010" z_local="0.020" material="mz_red"/>
+    <xacro:mz_cube name="cube_01" x_local="0.050" y_local="0.010" z_local="0.020" material="mz_green"/>
+    <xacro:mz_cube name="cube_02" x_local="0.090" y_local="0.010" z_local="0.020" material="mz_blue"/>
+    <xacro:mz_cube name="cube_10" x_local="0.010" y_local="0.050" z_local="0.020" material="mz_yellow"/>
+    <xacro:mz_cube name="cube_11" x_local="0.050" y_local="0.050" z_local="0.020" material="mz_orange"/>
+    <xacro:mz_cube name="cube_12" x_local="0.090" y_local="0.050" z_local="0.020" material="mz_white"/>
+    <xacro:mz_cube name="cube_20" x_local="0.010" y_local="0.090" z_local="0.020" material="mz_magenta"/>
+    <xacro:mz_cube name="cube_21" x_local="0.050" y_local="0.090" z_local="0.020" material="mz_cyan"/>
+    <xacro:mz_cube name="cube_22" x_local="0.090" y_local="0.090" z_local="0.020" material="mz_dark_gray"/>
   </xacro:macro>
 </robot>
