Commit message: Phase 1.1: realign layout to EstacionMezzanine.dxf
DXF (mm, INSUNITS=4) is now the source of truth for all planar XY positions.
Z values come from prior physical measurements or component specs where the
DXF does not provide height. Origin convention (table LL corner) unchanged.

Layout changes:
- conveyor: pos (0.500,0.300)->(0.385,0.302); size 0.400x0.132x0.055 ->
  0.700x0.215x0.060 (DOBOT Conveyor Belt Kit official).
- cube_base: pos (0.110,0.030)->(0.020,0.348); now upper-left of cobot.
- cubes: single demo cube replaced with 3x3 grid of 9 color-differentiated
  cubes (red/green/blue/yellow/orange/white/magenta/cyan/dark_gray) +
  5 mm reborde frame on the base.
- hmi: pos (0.650,0.425)->(0.650,0.517) (between conveyor back edge and
  PLC cabinet); base footprint 0.140x0.060 -> 0.168x0.067 per DXF.
- computer: pos (1.250,0.030)->(1.137,0.260); footprint now 0.372x0.432
  (full workstation area, extends past table edges). Tower (Lenovo tinker
  bbox 0.11825x0.07239x0.0861) at back-right; monitor + keyboard + mouse
  placeholders in front.
- photoelectric_sensor: local (0.210,0.120,0.050)->(0.217,0.218,0.060);
  now at back edge of conveyor per DXF U-shape bracket.
- camera_profile: column profile_x 0.690->0.598; arm length 0.316->0.169
  (exact recompute) so camera body centers over DXF orange footprint
  (0.618, 0.407, 0.635). Z kept from Phase 1.
- white_board: pos (0.090,0.035)->(0.109,0.034); kept as flat plate.
- cobot_base, plc_cabinet, buttons_panel: XY unchanged (DXF confirms).

New: explicit start_button (r=0.019) and emergency_stop_button (r=0.029)
positions per DXF circles. Materials add mz_magenta, mz_cyan,
mz_cube_base_brown.

Added reference/dxf/EstacionMezzanine.dxf and reference/rviz_screenshots/
phase_1_1_dxf_driven.png. docs/measurements.md gains the color-to-component
map and a Phase 1 -> 1.1 delta table; docs/validation.md updated with the
new expected coordinates.

Co-Authored-By: Claude Opus 4.7 (1M context) <noreply@anthropic.com>

File: mezzanine_rviz_sim/urdf/hmi.xacro (robot description, xacro)
@@ -7,11 +7,11 @@
       - hmi_display (the tilted display housing with screen)
     Display is tilted backward ~15 deg for operator viewing.
-    Position xyz = (0.650, 0.425, 0) m is the lower-left-front corner
-    of the base on the tabletop.
-    Dimensions are placeholders consistent with a 7" SIMATIC panel.
+    Position from EstacionMezzanine.dxf: LL = (0.650, 0.517, 0) m
+    (between conveyor back edge and PLC cabinet front edge).
+    Base footprint (0.168 x 0.067) matches the DXF rectangle (light blue).
   -->
-  <!-- Base + support -->
-  <xacro:property name="hmi_base_x" value="0.140"/>
-  <xacro:property name="hmi_base_y" value="0.060"/>
+  <!-- Base + support; base XY matches DXF footprint -->
+  <xacro:property name="hmi_base_x" value="0.168"/>
+  <xacro:property name="hmi_base_y" value="0.067"/>
   <xacro:property name="hmi_base_z" value="0.012"/>
   <xacro:property name="hmi_arm_x" value="0.030"/>
@@ -28,5 +28,5 @@
   <xacro:property name="hmi_tilt_deg" value="15"/>
   <xacro:property name="hmi_tilt_rad" value="${hmi_tilt_deg * 3.14159265 / 180}"/>
-  <xacro:macro name="mz_hmi" params="parent:=table_origin x:=0.650 y:=0.425 z:=0.000">
+  <xacro:macro name="mz_hmi" params="parent:=table_origin x:=0.650 y:=0.517 z:=0.000">
     <!-- hmi_panel: base plate + small support arm (Siemens beige/light gray) -->
     <link name="hmi_panel">

File: mezzanine_rviz_sim/urdf/materials.xacro (robot description, xacro)
@@ -43,3 +43,12 @@
     <color rgba="0.95 0.80 0.10 1.0"/>
   </material>
+  <material name="mz_magenta">
+    <color rgba="0.85 0.10 0.85 1.0"/>
+  </material>
+  <material name="mz_cyan">
+    <color rgba="0.10 0.85 0.85 1.0"/>
+  </material>
+  <material name="mz_cube_base_brown">
+    <color rgba="0.804 0.412 0.157 1.0"/>
+  </material>
 </robot>

File: mezzanine_rviz_sim/urdf/mezzanine_cell.urdf.xacro (robot description, xacro)
@@ -48,37 +48,44 @@
                           base_x="1.300" base_y="0.010" base_z="-0.720"/>
   <xacro:mz_plc_cabinet parent="table_origin" x="0.050" y="0.596" z="-0.073"/>
-  <xacro:mz_white_board parent="table_origin" x="0.090" y="0.035" z="0.000"/>
+  <!-- White board / flat plate (red rect in DXF, LL=(0.109, 0.034)) -->
+  <xacro:mz_white_board parent="table_origin" x="0.109" y="0.034" z="0.000"/>
   <!--
-    cube_base: revised to left-of-cobot per user feedback (was 0.348, 0.020).
-    Cobot center at x=0.240; cubes now sit at x=0.110 (left side, front edge).
-    TBD: confirm against physical layout in Phase 2.
+    cube_base (orange RGB 205,105,40 in DXF, LL=(0.020, 0.348)):
+    140x140 outer with 5 mm reborde and 9 cubes in a 3x3 grid (DXF yellow).
+    Cubes are color-differentiated (red, green, blue, yellow, orange, white,
+    magenta, cyan, dark_gray).
   -->
-  <xacro:mz_cube_base parent="table_origin" x="0.110" y="0.030" z="0.000"/>
+  <xacro:mz_cube_base parent="table_origin" x="0.020" y="0.348" z="0.000"/>
   <!--
-    Conveyor: revised to be further right per user feedback (was x=0.385).
-    Now at x=0.500. With 0.400 m length placeholder it extends 0.500..0.900.
-    TBD: confirm exact length and x against physical layout.
+    Conveyor (DOBOT Conveyor Belt Kit, blue in DXF, LL=(0.385, 0.302)):
+    official dimensions 0.700 x 0.215 x 0.060 m.
   -->
-  <xacro:mz_conveyor parent="table_origin" x="0.500" y="0.300" z="0.000"/>
+  <xacro:mz_conveyor parent="table_origin" x="0.385" y="0.302" z="0.000"/>
+  <!--
+    Photoelectric sensor body (cream RGB 248,246,176 U-shape in DXF):
+    center world (0.617, 0.530, ~0.060); local on conveyor_base = (0.217, 0.218, 0.060).
+  -->
   <xacro:mz_photoelectric_sensor parent="conveyor_base"
-                                 x="0.210" y="0.120" z="0.050"/>
+                                 x="0.217" y="0.218" z="0.060"/>
   <!--
-    Camera support: vertical column moved to back edge (pegado a la cabina)
-    per user feedback. profile_y=0.556 puts the column right behind the
-    PLC cabinet zone; arm length 0.316 m brings camera over the sensor area
-    at (~0.710, ~0.260, 0.635).
+    Camera support: column at LL=(0.598, 0.556) (pegada a la cabina, back edge),
+    arm 0.169 m in -y so the camera sits centered over the DXF orange
+    footprint (0.618, 0.407). Z=0.635 m kept from Phase 1 (DXF gives planar XY only).
   -->
   <xacro:mz_camera_support parent="table_origin"
-                           profile_x="0.690" profile_y="0.556"
-                           profile_arm_len_y="0.316"
+                           profile_x="0.598" profile_y="0.556"
+                           profile_arm_len_y="0.169"
                            camera_z="0.635"/>
-  <xacro:mz_hmi parent="table_origin" x="0.650" y="0.425" z="0.000"/>
+  <!-- HMI (light blue RGB 122,175,223 in DXF, LL=(0.650, 0.517)) -->
+  <xacro:mz_hmi parent="table_origin" x="0.650" y="0.517" z="0.000"/>
+  <!-- Start/E-Stop panel (cyan in DXF, LL=(1.170, 0.040)) -->
   <xacro:mz_buttons_panel parent="table_origin"
                           x="1.170" y="0.040" z="0.000"/>
   <!--
-    Computer: TBD position - placed at right side of the table per user
-    feedback. Tower + monitor placeholder.
+    Computer workstation footprint (magenta in DXF, LL=(1.137, 0.260)):
+    372 x 432 mm visual approximation containing tower + monitor + keyboard + mouse.
+    Footprint extends past the table edges (X: 1.137..1.509, Y: 0.260..0.692).
   -->
-  <xacro:mz_computer parent="table_origin" x="1.250" y="0.030" z="0.000"/>
+  <xacro:mz_computer parent="table_origin" x="1.137" y="0.260" z="0.000"/>
   <!--
     cobot_base: EXCEPTION to the lower-left-corner convention.

File: mezzanine_rviz_sim/urdf/photoelectric_sensor.xacro (robot description, xacro)
@@ -2,6 +2,10 @@
 <robot xmlns:xacro="http://ros.org/wiki/xacro">
   <!--
-    Photoelectric sensor. Dimensions are placeholders (TBD).
-    Reported (21, 12, 5) cm is treated as LOCAL to the conveyor.
+    Photoelectric sensor. Body box 0.030 x 0.020 x 0.040 m.
+    DXF source: U-shaped bracket (cream RGB 248,246,176) at conveyor back edge.
+    Body center (world frame): (0.617, 0.530, ~0.060). Conveyor_base local frame
+    has LL world (0.385, 0.302, 0), so local LL = (0.217, 0.218, 0.060).
+    Z = 0.060 rests the body on the conveyor top surface; the actual bracket
+    lifts it slightly higher - exact height TBD until physical measurement.
     The sensor is attached as child of conveyor_base.
   -->
@@ -9,5 +13,5 @@
   <xacro:property name="ps_size_y" value="0.020"/>
   <xacro:property name="ps_size_z" value="0.040"/>
-  <xacro:macro name="mz_photoelectric_sensor" params="parent:=conveyor_base x:=0.210 y:=0.120 z:=0.050">
+  <xacro:macro name="mz_photoelectric_sensor" params="parent:=conveyor_base x:=0.217 y:=0.218 z:=0.060">
     <link name="photoelectric_sensor">
       <visual>

File: mezzanine_rviz_sim/urdf/white_board.xacro (robot description, xacro)
@@ -2,12 +2,12 @@
 <robot xmlns:xacro="http://ros.org/wiki/xacro">
   <!--
-    White board / working plate.
-    Size 0.303 x 0.227 x 0.020 m. Position xyz = (0.090, 0.035, 0) m is
-    the lower-left-front corner on the tabletop.
+    White board / working plate (red rectangle in EstacionMezzanine.dxf).
+    Flat plate on the tabletop (horizontal, NOT a vertical board).
+    Size 0.303 x 0.227 x 0.020 m. Position from DXF: LL = (0.109, 0.034, 0) m.
   -->
   <xacro:property name="wb_size_x" value="0.303"/>
   <xacro:property name="wb_size_y" value="0.227"/>
   <xacro:property name="wb_size_z" value="0.020"/>
-  <xacro:macro name="mz_white_board" params="parent:=table_origin x:=0.090 y:=0.035 z:=0.000">
+  <xacro:macro name="mz_white_board" params="parent:=table_origin x:=0.109 y:=0.034 z:=0.000">
     <link name="white_board">
       <visual>
