Commit message: Adjust layout per user visual feedback (5 changes)
1. cube_base: moved from (0.348, 0.020) to (0.110, 0.030) - now on the
   left side of the cobot, per user feedback ("eso estaba a la izquierda
   del cobot").

2. conveyor: moved from x=0.385 to x=0.500 - shifted right per user
   feedback ("el conveyor lo veo que esta mas pegado a la izquierda,
   cuando deberia ir mas a la derecha"). Length 0.400 m still TBD.

3. Camera support: vertical column moved from (0.575, 0.400) to
   (0.690, 0.556) - now adjacent to the back edge, pegado a la cabina
   PLC, per user feedback. Horizontal arm length extended from 0.180 to
   0.316 m so the camera lands at the expected (0.710, 0.260, 0.635).
   profile_arm_len_y is now a macro parameter.

4. HMI: redesigned with Siemens KTP700 7" look - multi-visual link with
   a base plate, small upright support arm, and a tilted display housing
   (~15 deg backward) with a darker screen face. Replaces the prior
   single dark box. Position unchanged at (0.650, 0.425, 0).

5. computer: NEW component added at (1.250, 0.030, 0) on the right side
   of the table per user feedback ("pon la computadora a la derecha de
   la mesa"). Placeholder workstation: vertical tower + monitor with
   stand and screen face. Dimensions TBD.

Validated:
- catkin_make succeeded.
- xacro parses to 921-line URDF without new errors.
- TF spot-checks confirm new positions:
    world->cube_base    (0.110, 0.030, 0.000)
    world->conveyor_base(0.500, 0.300, 0.000)
    world->camera_frame (0.710, 0.260, 0.635)
    world->computer     (1.250, 0.030, 0.000)
- Updated screenshot at docs/screenshots/rviz_v2_layout_revised.png.

Co-Authored-By: Claude Opus 4.7 (1M context) <noreply@anthropic.com>

File: mezzanine_rviz_sim/urdf/camera_frame.xacro (robot description, xacro)
@@ -10,5 +10,4 @@
   <xacro:property name="profile_cs_y" value="0.040"/>
   <xacro:property name="profile_vertical_len" value="0.720"/>
-  <xacro:property name="profile_arm_len_y" value="0.180"/>
   <xacro:property name="camera_size_x" value="0.060"/>
   <xacro:property name="camera_size_y" value="0.060"/>
@@ -17,4 +16,5 @@
                                                  profile_x:=0.575
                                                  profile_y:=0.400
+                                                 profile_arm_len_y:=0.180
                                                  camera_z:=0.635">
     <link name="camera_profile">

File: mezzanine_rviz_sim/urdf/hmi.xacro (robot description, xacro)
@@ -2,23 +2,59 @@
 <robot xmlns:xacro="http://ros.org/wiki/xacro">
   <!--
-    HMI placeholder: 0.20 x 0.05 x 0.15 m (TBD).
-    Position xyz = (0.650, 0.425, 0) m is the lower-left-front corner.
+    HMI - Siemens SIMATIC HMI 7" (e.g. KTP700 Basic look).
+    Multi-link:
+      - hmi_panel (base + small support arm on the table)
+      - hmi_display (the tilted display housing with screen)
+    Display is tilted backward ~15 deg for operator viewing.
+    Position xyz = (0.650, 0.425, 0) m is the lower-left-front corner
+    of the base on the tabletop.
+    Dimensions are placeholders consistent with a 7" SIMATIC panel.
   -->
-  <xacro:property name="hmi_size_x" value="0.200"/>
-  <xacro:property name="hmi_size_y" value="0.050"/>
-  <xacro:property name="hmi_size_z" value="0.150"/>
+  <!-- Base + support -->
+  <xacro:property name="hmi_base_x" value="0.140"/>
+  <xacro:property name="hmi_base_y" value="0.060"/>
+  <xacro:property name="hmi_base_z" value="0.012"/>
+  <xacro:property name="hmi_arm_x" value="0.030"/>
+  <xacro:property name="hmi_arm_y" value="0.040"/>
+  <xacro:property name="hmi_arm_z" value="0.080"/>
+  <!-- Display housing (Siemens 7" KTP700: ~214 x 41 x 158 mm) -->
+  <xacro:property name="hmi_disp_x" value="0.214"/>
+  <xacro:property name="hmi_disp_y" value="0.041"/>
+  <xacro:property name="hmi_disp_z" value="0.158"/>
+  <!-- Active screen area (smaller than bezel) -->
+  <xacro:property name="hmi_scr_x" value="0.160"/>
+  <xacro:property name="hmi_scr_y" value="0.004"/>
+  <xacro:property name="hmi_scr_z" value="0.105"/>
+  <xacro:property name="hmi_tilt_deg" value="15"/>
+  <xacro:property name="hmi_tilt_rad" value="${hmi_tilt_deg * 3.14159265 / 180}"/>
   <xacro:macro name="mz_hmi" params="parent:=table_origin x:=0.650 y:=0.425 z:=0.000">
+    <!-- hmi_panel: base plate + small support arm (Siemens beige/light gray) -->
     <link name="hmi_panel">
+      <!-- base plate on the table -->
       <visual>
-        <origin xyz="${hmi_size_x/2} ${hmi_size_y/2} ${hmi_size_z/2}" rpy="0 0 0"/>
+        <origin xyz="${hmi_base_x/2} ${hmi_base_y/2} ${hmi_base_z/2}" rpy="0 0 0"/>
         <geometry>
-          <box size="${hmi_size_x} ${hmi_size_y} ${hmi_size_z}"/>
+          <box size="${hmi_base_x} ${hmi_base_y} ${hmi_base_z}"/>
         </geometry>
-        <material name="mz_hmi_dark"/>
+        <material name="mz_aluminum"/>
       </visual>
       <collision>
-        <origin xyz="${hmi_size_x/2} ${hmi_size_y/2} ${hmi_size_z/2}" rpy="0 0 0"/>
+        <origin xyz="${hmi_base_x/2} ${hmi_base_y/2} ${hmi_base_z/2}" rpy="0 0 0"/>
         <geometry>
-          <box size="${hmi_size_x} ${hmi_size_y} ${hmi_size_z}"/>
+          <box size="${hmi_base_x} ${hmi_base_y} ${hmi_base_z}"/>
+        </geometry>
+      </collision>
+      <!-- upright support arm at back-center of the base -->
+      <visual>
+        <origin xyz="${hmi_base_x/2} ${hmi_base_y - hmi_arm_y/2} ${hmi_base_z + hmi_arm_z/2}" rpy="0 0 0"/>
+        <geometry>
+          <box size="${hmi_arm_x} ${hmi_arm_y} ${hmi_arm_z}"/>
+        </geometry>
+        <material name="mz_aluminum"/>
+      </visual>
+      <collision>
+        <origin xyz="${hmi_base_x/2} ${hmi_base_y - hmi_arm_y/2} ${hmi_base_z + hmi_arm_z/2}" rpy="0 0 0"/>
+        <geometry>
+          <box size="${hmi_arm_x} ${hmi_arm_y} ${hmi_arm_z}"/>
         </geometry>
       </collision>
@@ -29,4 +65,41 @@
       <origin xyz="${x} ${y} ${z}" rpy="0 0 0"/>
     </joint>
+    <!-- hmi_display: the Siemens panel; tilted backward (rpy x) -->
+    <link name="hmi_display">
+      <!-- bezel / casing -->
+      <visual>
+        <origin xyz="0 0 0" rpy="0 0 0"/>
+        <geometry>
+          <box size="${hmi_disp_x} ${hmi_disp_y} ${hmi_disp_z}"/>
+        </geometry>
+        <material name="mz_panel_white"/>
+      </visual>
+      <collision>
+        <origin xyz="0 0 0" rpy="0 0 0"/>
+        <geometry>
+          <box size="${hmi_disp_x} ${hmi_disp_y} ${hmi_disp_z}"/>
+        </geometry>
+      </collision>
+      <!-- screen face on front (=-y of the display in display local frame) -->
+      <visual>
+        <origin xyz="0 ${-hmi_disp_y/2 - hmi_scr_y/2} 0" rpy="0 0 0"/>
+        <geometry>
+          <box size="${hmi_scr_x} ${hmi_scr_y} ${hmi_scr_z}"/>
+        </geometry>
+        <material name="mz_hmi_dark"/>
+      </visual>
+    </link>
+    <!--
+      Place hmi_display centered above the support arm, tilted backward ~15 deg
+      (rotating about world x so that the screen face leans toward the operator).
+    -->
+    <joint name="hmi_panel_to_hmi_display" type="fixed">
+      <parent link="hmi_panel"/>
+      <child link="hmi_display"/>
+      <origin xyz="${hmi_base_x/2}
+                   ${hmi_base_y - hmi_arm_y/2 + hmi_disp_y/2 * 0.5}
+                   ${hmi_base_z + hmi_arm_z + hmi_disp_z/2 - 0.010}"
+              rpy="${hmi_tilt_rad} 0 0"/>
+    </joint>
   </xacro:macro>
 </robot>

File: mezzanine_rviz_sim/urdf/mezzanine_cell.urdf.xacro (robot description, xacro)
@@ -34,4 +34,5 @@
   <xacro:include filename="$(find mezzanine_rviz_sim)/urdf/white_board.xacro"/>
   <xacro:include filename="$(find mezzanine_rviz_sim)/urdf/gripper_adapter.xacro"/>
+  <xacro:include filename="$(find mezzanine_rviz_sim)/urdf/computer.xacro"/>
   <link name="world"/>
   <link name="table_origin"/>
@@ -48,14 +49,36 @@
   <xacro:mz_plc_cabinet parent="table_origin" x="0.050" y="0.596" z="-0.073"/>
   <xacro:mz_white_board parent="table_origin" x="0.090" y="0.035" z="0.000"/>
-  <xacro:mz_cube_base parent="table_origin" x="0.348" y="0.020" z="0.000"/>
-  <xacro:mz_conveyor parent="table_origin" x="0.385" y="0.300" z="0.000"/>
+  <!--
+    cube_base: revised to left-of-cobot per user feedback (was 0.348, 0.020).
+    Cobot center at x=0.240; cubes now sit at x=0.110 (left side, front edge).
+    TBD: confirm against physical layout in Phase 2.
+  -->
+  <xacro:mz_cube_base parent="table_origin" x="0.110" y="0.030" z="0.000"/>
+  <!--
+    Conveyor: revised to be further right per user feedback (was x=0.385).
+    Now at x=0.500. With 0.400 m length placeholder it extends 0.500..0.900.
+    TBD: confirm exact length and x against physical layout.
+  -->
+  <xacro:mz_conveyor parent="table_origin" x="0.500" y="0.300" z="0.000"/>
   <xacro:mz_photoelectric_sensor parent="conveyor_base"
                                  x="0.210" y="0.120" z="0.050"/>
+  <!--
+    Camera support: vertical column moved to back edge (pegado a la cabina)
+    per user feedback. profile_y=0.556 puts the column right behind the
+    PLC cabinet zone; arm length 0.316 m brings camera over the sensor area
+    at (~0.710, ~0.260, 0.635).
+  -->
   <xacro:mz_camera_support parent="table_origin"
-                           profile_x="0.575" profile_y="0.400"
+                           profile_x="0.690" profile_y="0.556"
+                           profile_arm_len_y="0.316"
                            camera_z="0.635"/>
   <xacro:mz_hmi parent="table_origin" x="0.650" y="0.425" z="0.000"/>
   <xacro:mz_buttons_panel parent="table_origin"
                           x="1.170" y="0.040" z="0.000"/>
+  <!--
+    Computer: TBD position - placed at right side of the table per user
+    feedback. Tower + monitor placeholder.
+  -->
+  <xacro:mz_computer parent="table_origin" x="1.250" y="0.030" z="0.000"/>
   <!--
     cobot_base: EXCEPTION to the lower-left-corner convention.

Commit message: Phase 1.2: world=floor, camera mounted to PLC cabinet, xArm home pose, aluminum gripper
Visual cleanup pass over the Phase 1.1 layout. No DXF XY changes; only the
vertical frame hierarchy, the camera support parenting, the xArm initial
pose, and the gripper materials.

Hierarchy changes:
- world now represents the real floor; the RViz grid renders at z = 0.
- table_origin is a child of world, elevated 0.746 m so the tabletop sits
  on the supports above the floor (support base 0.030 + column 0.690 +
  tabletop 0.026).
- Table support bases now rest on the floor (table_origin z = -0.746
  instead of -0.720).
- New frame plc_cabinet_camera_mount on the cabinet top, front face, at
  local (0.548, 0, 0). camera_profile is parented here so the aluminum
  column rises visibly from the cabinet rather than floating mid-table.
  The arm extends -y by 0.209 m and the camera body still lands centered
  over the DXF orange footprint at world (0.618, 0.407, 1.381).

Visual / pose:
- xArm 6 home pose published via joint_state_publisher zeros rosparam:
  joint1=0.0, joint2=-0.6, joint3=-1.2, joint4=0.0, joint5=1.5, joint6=0.0.
- Gripper materials switched to aluminum tones:
    gripper_base = aluminum_dark
    gripper_body = aluminum_light
    fingers      = brushed_aluminum
  Added aluminum_light/dark/brushed_aluminum in materials.xacro.
- rviz/mezzanine.rviz: orbit Distance 2.5->3.5, Focal Point Z 0->0.75,
  Pitch 0.6->0.5, Yaw 4.5->4.6; side docks collapsed so the 3D viewport
  takes the full window.

New screenshot: docs/screenshots/rviz_world_floor_camera_mount_gripper_home.png.

Co-Authored-By: Claude Opus 4.7 (1M context) <noreply@anthropic.com>

File: mezzanine_rviz_sim/urdf/camera_frame.xacro (robot description, xacro)
@@ -2,25 +2,36 @@
 <robot xmlns:xacro="http://ros.org/wiki/xacro">
   <!--
-    Camera support: vertical aluminum profile (4x4 cm cross section) standing
-    at LL=(0.598, 0.556) m (pegada a la cabina - back edge at y=0.596),
-    with a horizontal arm extending in -y to support the camera.
-    DXF source: orange RGB 248,153,30 rectangle (camera body footprint
-    centered at (0.618, 0.407)).
-    Geometry: camera_world_y = profile_y + cs_y/2 - arm_len_y. With
-    profile_y=0.556, cs_y/2=0.020 and camera_y=0.407, arm_len_y=0.169 m
-    (computed exact instead of 0.189 m estimate from the diagnostic).
-    Z=0.635 m kept from Phase 1; the DXF only provides planar XY.
+    Camera support: vertical aluminum profile (4x4 cm cross section)
+    mounted to the PLC cabinet top via the `plc_cabinet_camera_mount`
+    frame, with a horizontal arm extending in -y to hold the camera over
+    the DXF orange footprint (world XY = (0.618, 0.407)).
+    Default parent = plc_cabinet_camera_mount (child of plc_cabinet).
+    Mount world frame after the world=floor lift:
+      world XY = (0.598, 0.596)  (cabinet front face at column LL X)
+      world Z  = 0.673           (cabinet top surface = table_origin Z=-0.073)
+    With profile_x=profile_y=profile_z=0, the column LL coincides with the
+    mount, so the column body extends from the cabinet front face onto the
+    cabinet top (Y 0.596 to 0.636 in world) and rises in +Z.
+    Camera Z target: world Z = 1.381 (kept 0.635 m above the table top).
+    Because the column LL is now at world Z = 0.673 instead of 0.746,
+    camera_z (profile-local) = 1.381 - 0.673 = 0.708 m.
+    profile_vertical_len bumped to 0.768 m so the arm (at vertical_len - cs_y/2
+    = 0.748) sits above the camera with ~0.040 m margin.
+    Arm length to bring camera centre to world Y = 0.407:
+      world Y_arm_end = profile_y_world + cs_y/2 - arm_len_y
+      0.407 = 0.596 + 0.020 - arm_len_y -> arm_len_y = 0.209 m.
   -->
   <xacro:property name="profile_cs_x" value="0.040"/>
   <xacro:property name="profile_cs_y" value="0.040"/>
-  <xacro:property name="profile_vertical_len" value="0.720"/>
+  <xacro:property name="profile_vertical_len" value="0.768"/>
   <xacro:property name="camera_size_x" value="0.060"/>
   <xacro:property name="camera_size_y" value="0.060"/>
   <xacro:property name="camera_size_z" value="0.060"/>
-  <xacro:macro name="mz_camera_support" params="parent:=table_origin
-                                                 profile_x:=0.598
-                                                 profile_y:=0.556
-                                                 profile_arm_len_y:=0.169
-                                                 camera_z:=0.635">
+  <xacro:macro name="mz_camera_support" params="parent:=plc_cabinet_camera_mount
+                                                 profile_x:=0
+                                                 profile_y:=0
+                                                 profile_z:=0
+                                                 profile_arm_len_y:=0.209
+                                                 camera_z:=0.708">
     <link name="camera_profile">
       <!-- vertical aluminum column -->
@@ -56,5 +67,5 @@
       <parent link="${parent}"/>
       <child link="camera_profile"/>
-      <origin xyz="${profile_x} ${profile_y} 0" rpy="0 0 0"/>
+      <origin xyz="${profile_x} ${profile_y} ${profile_z}" rpy="0 0 0"/>
     </joint>
     <link name="camera_frame">

File: mezzanine_rviz_sim/urdf/gripper_adapter.xacro (robot description, xacro)
@@ -34,5 +34,5 @@
           <box size="${gb_size_x} ${gb_size_y} ${gb_size_z}"/>
         </geometry>
-        <material name="mz_dark_gray"/>
+        <material name="aluminum_dark"/>
       </visual>
       <collision>
@@ -54,5 +54,5 @@
           <box size="${body_size_x} ${body_size_y} ${body_size_z}"/>
         </geometry>
-        <material name="mz_dark_gray"/>
+        <material name="aluminum_light"/>
       </visual>
       <collision>
@@ -74,5 +74,5 @@
           <box size="${finger_thickness} ${finger_thickness} ${finger_height}"/>
         </geometry>
-        <material name="mz_dark_gray"/>
+        <material name="brushed_aluminum"/>
       </visual>
       <collision>
@@ -94,5 +94,5 @@
           <box size="${finger_thickness} ${finger_thickness} ${finger_height}"/>
         </geometry>
-        <material name="mz_dark_gray"/>
+        <material name="brushed_aluminum"/>
       </visual>
       <collision>

File: mezzanine_rviz_sim/urdf/materials.xacro (robot description, xacro)
@@ -52,3 +52,13 @@
     <color rgba="0.804 0.412 0.157 1.0"/>
   </material>
+  <!-- Aluminum tones for gripper and visual highlight surfaces -->
+  <material name="aluminum_light">
+    <color rgba="0.78 0.78 0.74 1.0"/>
+  </material>
+  <material name="aluminum_dark">
+    <color rgba="0.55 0.55 0.52 1.0"/>
+  </material>
+  <material name="brushed_aluminum">
+    <color rgba="0.70 0.70 0.66 1.0"/>
+  </material>
 </robot>

File: mezzanine_rviz_sim/urdf/mezzanine_cell.urdf.xacro (robot description, xacro)
@@ -35,4 +35,12 @@
   <xacro:include filename="$(find mezzanine_rviz_sim)/urdf/gripper_adapter.xacro"/>
   <xacro:include filename="$(find mezzanine_rviz_sim)/urdf/computer.xacro"/>
+  <!--
+    Frame hierarchy (Phase 1.2):
+      world         = real floor (RViz grid sits here, z=0)
+      table_origin  = lower-left corner of the tabletop top surface
+                      (elevated 0.746 m above the floor:
+                       support base 0.030 + column 0.690 + table 0.026).
+    All XY positions from the DXF stay expressed in the table_origin frame.
+  -->
   <link name="world"/>
   <link name="table_origin"/>
@@ -40,11 +48,16 @@
     <parent link="world"/>
     <child link="table_origin"/>
-    <origin xyz="0 0 0" rpy="0 0 0"/>
+    <origin xyz="0 0 0.746" rpy="0 0 0"/>
   </joint>
   <xacro:mz_table parent="table_origin"/>
+  <!--
+    Table supports: bases sit on the floor (world z=0 ≡ table_origin z=-0.746).
+    Column extends from base top (z=-0.716) to just below the tabletop
+    (z=-0.026). Tabletop occupies z=-0.026..0 in table_origin.
+  -->
   <xacro:mz_table_support side="left"  parent="table_origin"
-                          base_x="0.030" base_y="0.010" base_z="-0.720"/>
+                          base_x="0.030" base_y="0.010" base_z="-0.746"/>
   <xacro:mz_table_support side="right" parent="table_origin"
-                          base_x="1.300" base_y="0.010" base_z="-0.720"/>
+                          base_x="1.300" base_y="0.010" base_z="-0.746"/>
   <xacro:mz_plc_cabinet parent="table_origin" x="0.050" y="0.596" z="-0.073"/>
   <!-- White board / flat plate (red rect in DXF, LL=(0.109, 0.034)) -->
@@ -69,12 +82,12 @@
                                  x="0.217" y="0.218" z="0.060"/>
   <!--
-    Camera support: column at LL=(0.598, 0.556) (pegada a la cabina, back edge),
-    arm 0.169 m in -y so the camera sits centered over the DXF orange
-    footprint (0.618, 0.407). Z=0.635 m kept from Phase 1 (DXF gives planar XY only).
+    Camera support: aluminum profile parented to the cabinet front face via
+    `plc_cabinet_camera_mount`. Column rises from the cabinet top; arm extends
+    0.209 m in -y so the camera body centers over the DXF orange footprint
+    (world XY = (0.618, 0.407)). camera_z = 0.708 in profile-local frame
+    keeps the camera body at world Z = 1.381 (= table top 0.746 + 0.635).
+    Macro defaults already encode all of this; we just pass the parent.
   -->
-  <xacro:mz_camera_support parent="table_origin"
-                           profile_x="0.598" profile_y="0.556"
-                           profile_arm_len_y="0.169"
-                           camera_z="0.635"/>
+  <xacro:mz_camera_support parent="plc_cabinet_camera_mount"/>
   <!-- HMI (light blue RGB 122,175,223 in DXF, LL=(0.650, 0.517)) -->
   <xacro:mz_hmi parent="table_origin" x="0.650" y="0.517" z="0.000"/>

File: mezzanine_rviz_sim/urdf/plc_cabinet.xacro (robot description, xacro)
@@ -30,4 +30,21 @@
       <origin xyz="${x} ${y} ${z}" rpy="0 0 0"/>
     </joint>
+    <!--
+      Camera mount frame on the PLC cabinet top surface.
+      Position is LOCAL to plc_cabinet link (top-LL-front corner):
+        x = 0.548 -> world X = 0.598 (matches camera column LL X from DXF)
+        y = 0     -> cabinet front face (world Y = 0.596 = table back edge)
+        z = 0     -> cabinet TOP surface
+      The vertical aluminum profile that holds the camera is parented here,
+      so the column visibly rises from the cabinet top instead of floating
+      over the tabletop. Camera body still lands over the DXF footprint
+      center (world XY = (0.618, 0.407)).
+    -->
+    <link name="plc_cabinet_camera_mount"/>
+    <joint name="plc_cabinet_to_plc_cabinet_camera_mount" type="fixed">
+      <parent link="plc_cabinet"/>
+      <child link="plc_cabinet_camera_mount"/>
+      <origin xyz="0.548 0 0" rpy="0 0 0"/>
+    </joint>
   </xacro:macro>
 </robot>
